Commit message: V1.1
修复了：
1，差速驱动方向反向错误（轮子Z轴朝向错误）。
2，rviz和MBF的action通信桥接成功，现在可以直接在Rviz发送 nav 2D goal控制移动。
3，修复cost map全部free的Bug，但是还是不能自主导航

File: src/b2_robot_pkgs/models/tracked_robot/mid360_sensor.urdf.xacro (robot description, xacro)
@@ -60,5 +60,5 @@
     <parent link="base_link"/>
     <child link="livox_link"/>
-    <origin xyz="0.2 0.0 0.15" rpy="0 0 0"/>
+    <origin xyz="0.25 0.0 0.15" rpy="0 0 0"/>
   </joint>
   <joint name="imu_joint" type="fixed">
@@ -100,5 +100,5 @@
           <range>
             <min>0.1</min>
-            <max>50.0</max>
+            <max>40.0</max>
             <resolution>0.01</resolution>
           </range>
@@ -125,7 +125,7 @@
       </angular_velocity>
       <linear_acceleration>
-        <x><noise type="gaussian"><mean>0.0</mean><stddev>0.1</stddev></noise></x>
-        <y><noise type="gaussian"><mean>0.0</mean><stddev>0.1</stddev></noise></y>
-        <z><noise type="gaussian"><mean>0.0</mean><stddev>0.1</stddev></noise></z>
+        <x><noise type="gaussian"><mean>0.0</mean><stddev>0.01</stddev></noise></x>
+        <y><noise type="gaussian"><mean>0.0</mean><stddev>0.01</stddev></noise></y>
+        <z><noise type="gaussian"><mean>0.0</mean><stddev>0.01</stddev></noise></z>
       </linear_acceleration>
     </imu>
@@ -139,10 +139,12 @@
       <odometryTopic>odom_topic</odometryTopic>
       <robotBaseFrame>base_link</robotBaseFrame>
-      <leftJoint>right_track_joint</leftJoint>
-      <rightJoint>left_track_joint</rightJoint>
+      <leftJoint>left_track_joint</leftJoint>
+      <rightJoint>right_track_joint</rightJoint>
+      <!-- <leftJoint>right_track_joint</leftJoint>
+      <rightJoint>left_track_joint</rightJoint> -->
       <wheelSeparation>0.35</wheelSeparation>
       <wheelDiameter>0.15</wheelDiameter>
-      <maxWheelTorque>5</maxWheelTorque>
-      <maxWheelAcceleration>0.5</maxWheelAcceleration>
+      <maxWheelTorque>10</maxWheelTorque>
+      <maxWheelAcceleration>2.0</maxWheelAcceleration>
       <odometrySource>1</odometrySource>
       <publishOdomTF>false</publishOdomTF>
@@ -199,5 +201,5 @@
     <parent link="base_link"/>
     <child link="left_track_link"/>
-    <origin xyz="0.1 0.2 -0.1" rpy="1.5708 0 0"/>
+    <origin xyz="-0.1 0.2 -0.1" rpy="-1.5708 0 0"/>
     <axis xyz="0 0 1"/>
   </joint>
@@ -205,5 +207,5 @@
     <parent link="base_link"/>
     <child link="right_track_link"/>
-    <origin xyz="0.1 -0.2 -0.10" rpy="1.5708 0 0"/>
+    <origin xyz="-0.1 -0.2 -0.10" rpy="-1.5708 0 0"/>
     <axis xyz="0 0 1"/>
   </joint>
@@ -233,5 +235,5 @@
     <parent link="base_link"/>
     <child link="caster_wheel_h"/>
-    <origin xyz="-0.2 0 -0.1375" rpy="0 0 0"/>
+    <origin xyz="0.2 0 -0.1375" rpy="0 0 0"/>
   </joint>
   <gazebo reference="caster_wheel_h">
@@ -242,3 +244,12 @@
     <maxVel>0.01</maxVel>
   </gazebo>
+<gazebo reference="base_link">
+  <material>Gazebo/Red</material>
+</gazebo>
+<gazebo reference="left_track_link">
+  <material>Gazebo/Blue</material>
+</gazebo>
+<gazebo reference="right_track_link">
+  <material>Gazebo/Black</material>
+</gazebo>
 </robot>
